File: SmallKat Battery Charger.kicad_pcb (KiCad board)
At the start: 4 copper layers, 50 x 50 mm, 60 parts, among them J1 Conn_01x02_Male, J2 Conn_01x04_Male, J3 Conn_01x04_Male, J4 Conn_01x03_Male, J5 Conn_01x06_Male, J6 Conn_01x02_Male, J7 Conn_01x02_Male, Q1 BUK7M33-60EX, Q2 BUK7M33-60EX, Q4 DMP3013SFV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

Commit message: upated board layout
Parts:
- C1, C10, C12, C7, C9: value C -> 0.1uF
- C11: value C -> 0.33uF
- C15, C16, C3, C8: value C -> 1uF
- C2: value C -> 47nF
- C4, C5: value C -> 10uF
- C6: value C -> 200uF
- L1: value L -> 2.2uH
- R1, R10, R14, R19, R5, R8: value R -> 10k
- R11: value R -> 160
- R12: value R -> 260
- R13: value R -> 100k
- R15: value R -> 6.5k
- R16: value R -> 10m
- R17, R18: value R -> 100
- R2: value R -> 430k
- R20: value R -> 10
- R25, R26, R27: value R -> 330
- R3: value R -> 66.5k
- R4: value R -> 4k; moved to F.Cu
- R6: value R -> 4k
- R7: value R -> 10m; moved to F.Cu
- R9: value R -> 15
- U1: moved to F.Cu
- moved R7 11.7 mm to (12.7, 7.65), turned to 90 degrees
- moved U1 3.27 mm to (9.30, 7.85), turned to 180 degrees
- moved R4 0.72 mm to (7.60, 14.4), turned to 180 degrees
Connections:
- net Net-(C1-Pad1) renamed GATE
- net Net-(C1-Pad2) renamed SOURCE
- net Net-(C2-Pad1) renamed BTST
- net Net-(R19-Pad2) renamed OUT
- net Net-(R2-Pad2) renamed ACDET
- net Net-(R7-Pad2) renamed ACP
- C4 pad 1: ADAPTER -> ACN
- C6 pad 1: SRP -> GND
- C6 pad 2: GND -> SRP
- Q1 pad 5: ADAPTER -> ACN
- R7 pad 1: Net-(R7-Pad1) -> ACN
- U3 pad 1: Net-(R7-Pad1) -> ACN
Routing:
- net ACN: track 0.00 -> 12.7 mm, vias 0 -> 2
- net GATE: track 4.36 -> 15.2 mm
- net SOURCE: track 6.75 -> 15.1 mm, vias 0 -> 1
- net Net-(R7-Pad1): track 2.36 -> 0.00 mm
- net ADAPTER: track 6.43 -> 4.27 mm, vias 31 -> 1
- net ACP: track 10.6 -> 12.7 mm
- net Net-(R4-Pad1): track 1.51 -> 1.60 mm, vias 0 -> 1
- net GND: vias 144 -> 143
- added copper zone on F.Cu, net ACN
- added copper zone on F.Cu, net ACP
- removed copper zone on B.Cu, net ADAPTER

Commit message: updated footprints
Parts:
- removed C13, C14: C, Capacitor_SMD:C_0402_1005Metric
- C4, C5, C6: footprint Capacitor_SMD:C_0402_1005Metric -> Capacitor_SMD:C_0805_2012Metric
- moved C6 6.04 mm to (34.9, 7.60), turned to 180 degrees
- moved U1 1.15 mm to (9.20, 9.00)
- moved C4 1.09 mm to (16.3, 4.60)
- moved C5 0.60 mm to (33.8, 13.8)
Routing:
- net ACN: track 12.7 -> 15.9 mm
- net SRP: track 37.3 -> 39.8 mm
- net GATE: track 15.2 -> 14.0 mm
- net CS: track 31.4 -> 30.2 mm
- net ACP: track 12.7 -> 11.8 mm
- net GND: track 30.9 -> 30.5 mm, vias 143 -> 144
- net Net-(C10-Pad1): vias 2 -> 1
