File: SmallKat Battery Charger.sch (KiCad schematic (older format))
At the start: 58 parts, among them J1 Conn_01x02_Male, J2 Conn_01x04_Male, J3 Conn_01x04_Male, J4 Conn_01x03_Male, J5 Conn_01x06_Male, J6 Conn_01x02_Male, J7 Conn_01x02_Male, Q1 BUK7M33-60EX, Q2 BUK7M33-60EX, Q4 DMP3013SFV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

Commit message: upated board layout
Connections:
- net labels removed: RAC
Changed lines of the file:
@@
 Text GLabel 9000 3750 1    50   Input ~ 0
 ADAPTER
-Text GLabel 6300 2350 1    50   Input ~ 0
-RAC
 Wire Wire Line
 	8550 5050 8100 5050
@@
 Wire Wire Line
 	9300 2000 9300 2300
-Text GLabel 8450 1850 1    50   Input ~ 0
-RAC
-Text GLabel 6400 750  1    50   Input ~ 0
-RAC
-Text GLabel 6400 750  3    50   Input ~ 0
+Text GLabel 6300 2350 1    50   Input ~ 0
 ACN
 Text Notes 950  1500 0    50   ~ 0
@@
 Wire Notes Line
 	450  450  450  7150
+Text GLabel 8450 1850 1    50   Input ~ 0
+ACN
 $EndSCHEMATC

Commit message: updated footprints
Parts:
- C4, C5, C6: footprint Capacitor_SMD:C_0402_1005Metric -> Capacitor_SMD:C_0805_2012Metric
Changed lines of the file:
@@
 F 0 "C5" H 9065 2496 50  0000 L CNN
 F 1 "10uF" H 9065 2405 50  0000 L CNN
-F 2 "Capacitor_SMD:C_0402_1005Metric" H 8988 2300 50  0001 C CNN
+F 2 "Capacitor_SMD:C_0805_2012Metric" H 8988 2300 50  0001 C CNN
 F 3 "~" H 8950 2450 50  0001 C CNN
 	1    8950 2450
@@
 F 0 "C6" H 9565 2046 50  0000 L CNN
 F 1 "200uF" H 9565 1955 50  0000 L CNN
-F 2 "Capacitor_SMD:C_0402_1005Metric" H 9488 1850 50  0001 C CNN
+F 2 "Capacitor_SMD:C_0805_2012Metric" H 9488 1850 50  0001 C CNN
 F 3 "~" H 9450 2000 50  0001 C CNN
 	1    9450 2000
@@
 F 0 "C4" H 6415 2546 50  0000 L CNN
 F 1 "10uF" H 6415 2455 50  0000 L CNN
-F 2 "Capacitor_SMD:C_0402_1005Metric" H 6338 2350 50  0001 C CNN
+F 2 "Capacitor_SMD:C_0805_2012Metric" H 6338 2350 50  0001 C CNN
 F 3 "~" H 6300 2500 50  0001 C CNN
 	1    6300 2500
